File: Controllers/CD32/CD32_Controller.sch (KiCad schematic (older format))
At the start: 24 parts, among them IC1 74LS165, IC2 74LS125, J1 DB9, SW1 Up, SW2 Down, SW3 Left, SW4 Right

Commit message: Added Atari Jaguar controller
Parts:
- removed RA1: 10K, Resistors_THT:R_Array_SIP10, symbol R_Network09
- added R10, R11, R12, R3, R4, R6, R7, R8, R9: 10K, Resistors_THT:R_Axial_DIN0207_L6.3mm_D2.5mm_P10.16mm_Horizontal, symbol Device:R
- C1: value C -> 220uF; footprint (none) -> Capacitors_THT:CP_Radial_D6.3mm_P2.50mm; symbol C -> Device:C
- C2: footprint (none) -> Capacitors_THT:CP_Radial_D6.3mm_P2.50mm; symbol CP -> Device:CP
- C3, C4: value C -> 100n; footprint (none) -> Capacitors_THT:C_Axial_L5.1mm_D3.1mm_P7.50mm_Horizontal; symbol C -> Device:C
- C5: renamed from C4; footprint (none) -> Capacitors_THT:C_Axial_L5.1mm_D3.1mm_P7.50mm_Horizontal; symbol C -> Device:C
- IC1: footprint (none) -> Housings_DIP:DIP-16_W7.62mm_LongPads; symbol 74LS165 -> CD32_Controller-rescue:74LS165
- IC2: footprint (none) -> Housings_DIP:DIP-14_W7.62mm_LongPads; symbol 74LS125 -> CD32_Controller-rescue:74LS125
- J1: footprint (none) -> Connector_Dsub:DSUB-9_Male_Horizontal_P2.77x2.84mm_EdgePinOffset4.94mm_Housed_MountingHolesOffset7.48mm; symbol DB9_Female -> CD32_Controller-rescue:DB9_Female
- L1: footprint (none) -> Inductors_THT:L_Axial_L5.3mm_D2.2mm_P10.16mm_Horizontal_Vishay_IM-1; symbol L -> Device:L
- R1, R2, R5: footprint (none) -> Resistors_THT:R_Axial_DIN0207_L6.3mm_D2.5mm_P10.16mm_Horizontal; symbol R -> Device:R
- SW1, SW2, SW3, SW4: footprint (none) -> Buttons_Switches_THT:SW_PUSH_6mm_h4.3mm; symbol SW_Push -> CD32_Controller-rescue:SW_Push
- SW10, SW11, SW5, SW6, SW7, SW8, SW9: renamed from SW?; footprint (none) -> Buttons_Switches_THT:SW_PUSH_6mm_h4.3mm; symbol SW_Push -> CD32_Controller-rescue:SW_Push
Connections:
- net GND: now also C1.2; no longer C1.1
- net VCC: now also R10.1, R11.1, R12.1, R3.1, R4.1, R6.1, R7.1, R8.1, R9.1
- net at IC1.2 (CP), IC2.11 (O), J1.6: now also R6.2
- net at J1.9, L1.2: now also C1.1; no longer C1.2
- net at C5.1, IC1.1 (Pl), IC2.6 (O): now also R3.2
- net at IC1.12 (P1), SW6.1: now also R4.2
- net at IC1.13 (P2), SW5.1: now also R7.2
- net at IC1.14 (P3), SW11.2: now also R8.2
- net at IC1.3 (P4), SW7.1: now also R9.2
- net at IC1.4 (P5), SW9.1: now also R10.2
- net at IC1.5 (P6), IC2.12 (D), SW8.1: now also R11.2
- net at IC1.6 (P7), SW10.1: now also R12.2
Other:
- note removed: "Pin 1 to VCC"
